Commit message: add cloning gazebo_ros_pkgs and catkin_make gazebo_ros and gazebo_ros_control folders

File: src/flexrobot_description_pkg/urdf/FlexRobotwSupporter_v3_2.xacro (robot description, xacro)
@@ -30,4 +30,10 @@
    </xacro:macro>
 -->
+  <!-- Used for fixing robot to Gazebo 'base_link' -->
+  <link name="world"/>
+  <joint name="fixed" type="fixed">
+    <parent link="world"/>
+    <child link="Supporter"/>
+  </joint>
   <link
     name="Supporter">
